Commit message: feat: adapt files to work with ignition

File: robots/borinot/xacro/definition.urdf.xacro (robot description, xacro)
@@ -5,5 +5,5 @@
   <xacro:include
     filename="$(find hidro_robots)/robots/common/xacro/sensors.xacro" />
-  <xacro:macro name="borinot_platform" params="robot_name simulation event_based_sim has_arm">
+  <xacro:macro name="borinot_platform" params="robot_name simulation simulation_sync simulation_px4 has_arm">
     <xacro:property name="platform_name" value="borinot" />
     <!-- platform -->
@@ -44,5 +44,5 @@
       direction="cw"
       simulation="${simulation}"
-      event_based_sim="${event_based_sim}"
+      simulation_px4="${simulation_px4}"
     />
     <xacro:rotor
@@ -55,5 +55,5 @@
       direction="ccw"
       simulation="${simulation}"
-      event_based_sim="${event_based_sim}"
+      simulation_px4="${simulation_px4}"
     />
     <xacro:rotor
@@ -66,5 +66,5 @@
       direction="cw"
       simulation="${simulation}"
-      event_based_sim="${event_based_sim}"
+      simulation_px4="${simulation_px4}"
     />
     <xacro:rotor
@@ -77,5 +77,5 @@
       direction="ccw"
       simulation="${simulation}"
-      event_based_sim="${event_based_sim}"
+      simulation_px4="${simulation_px4}"
     />
     <xacro:rotor
@@ -88,5 +88,5 @@
       direction="ccw"
       simulation="${simulation}"
-      event_based_sim="${event_based_sim}"
+      simulation_px4="${simulation_px4}"
     />
     <xacro:rotor
@@ -99,8 +99,8 @@
       direction="cw"
       simulation="${simulation}"
-      event_based_sim="${event_based_sim}"
+      simulation_px4="${simulation_px4}"
     />
     <xacro:if value="${simulation}">
-      <xacro:unless value="${event_based_sim}">
+      <xacro:if value="${simulation_px4}">
         <xacro:px4_plugins
           robot_name="${robot_name}"
@@ -183,5 +183,5 @@
           </plugin>
         </gazebo>
-      </xacro:unless>
+      </xacro:if>
     </xacro:if>
   </xacro:macro>

File: robots/borinot/xacro/description.urdf.xacro (robot description, xacro)
@@ -9,19 +9,72 @@
   <!-- arguments -->
   <xacro:arg name="simulation" default="true" />
-  <xacro:arg name="event_based_sim" default="false" />
+  <xacro:arg name="simulation_sync" default="false" />
+  <xacro:arg name="simulation_px4" default="false" />
   <!-- properties -->
   <xacro:property name="simulation" value="$(arg simulation)" />
-  <xacro:property name="event_based_sim" value="$(arg event_based_sim)" />
+  <xacro:property name="simulation_sync" value="$(arg simulation_sync)" />
+  <xacro:property name="simulation_px4" value="$(arg simulation_px4)" />
+  <xacro:if value="${simulation_sync}">
+    <xacro:property name="simulation_px4" value="false" />
+  </xacro:if>
   <xacro:borinot_platform
     robot_name="borinot"
     simulation="${simulation}"
-    event_based_sim="${event_based_sim}"
+    simulation_sync="${simulation_sync}"
+    simulation_px4="${simulation_px4}"
     has_arm="false"
   />
   <xacro:if value="${simulation}">
-    <xacro:if value="${event_based_sim}">
+    <xacro:if value="${simulation_sync}">
       <gazebo>
+        <plugin name='eagle_ros2_gz::EagleGzSyncSimPlugin'
+          filename='libeagle_gz_sync_sim_plugin.so'>
+          <simulationRate>2000</simulationRate>
+          <actuationRate>500</actuationRate>
+          <ramStateTopic>/borinot/uam_state</ramStateTopic>
+          <ramControlTopic>/borinot/uam_control</ramControlTopic>
+          <platform_params>
+            <baselinkName>borinot__base_link</baselinkName>
+            <thrustToTorqueRatio>0.01393568</thrustToTorqueRatio>
+            <thrustBias>1.0</thrustBias>
+            <rotor_params>
+              <number>0</number>
+              <linkName>borinot__rotor0</linkName>
+              <turningDirection>-1</turningDirection>
+            </rotor_params>
+            <rotor_params>
+              <number>1</number>
+              <linkName>borinot__rotor1</linkName>
+              <turningDirection>1</turningDirection>
+            </rotor_params>
+            <rotor_params>
+              <number>2</number>
+              <linkName>borinot__rotor2</linkName>
+              <turningDirection>-1</turningDirection>
+            </rotor_params>
+            <rotor_params>
+              <number>3</number>
+              <linkName>borinot__rotor3</linkName>
+              <turningDirection>1</turningDirection>
+            </rotor_params>
+            <rotor_params>
+              <number>4</number>
+              <linkName>borinot__rotor4</linkName>
+              <turningDirection>1</turningDirection>
+            </rotor_params>
+            <rotor_params>
+              <number>5</number>
+              <linkName>borinot__rotor5</linkName>
+              <turningDirection>-1</turningDirection>
+            </rotor_params>
+          </platform_params>
+        </plugin>
+      </gazebo>
+    </xacro:if>
+    <xacro:unless value="${simulation_sync}">
+      <xacro:unless value="${simulation_px4}">
+        <!-- <gazebo>
         <plugin name='eagle_gazebo_event_base_sim_plugin'
-          filename='libeagle_gazebo_event_based_sim_plugin.so'>
+          filename='libeagle_gazebo_simulation_sync_plugin.so'>
           <simulationRate>2000</simulationRate>
           <actuationRate>500</actuationRate>
@@ -62,8 +115,8 @@
             </rotor_params>
           </platform_params>
-          <!-- here add the arm -->
         </plugin>
-      </gazebo>
-    </xacro:if>
+      </gazebo> -->
+      </xacro:unless>
+    </xacro:unless>
   </xacro:if>
 </robot>

File: robots/borinot_flying_arm_2/xacro/description.urdf.xacro (robot description, xacro)
@@ -7,8 +7,8 @@
   <!-- arguments -->
   <xacro:arg name="simulation" default="true" />
-  <xacro:arg name="event_based_sim" default="false" />
+  <xacro:arg name="simulation_sync" default="false" />
   <!-- properties -->
   <xacro:property name="simulation" value="$(arg simulation)" />
-  <xacro:property name="event_based_sim" value="$(arg event_based_sim)" />
+  <xacro:property name="simulation_sync" value="$(arg simulation_sync)" />
   <xacro:property name="robot_name" value="borinot_flying_arm_2" />
   <xacro:borinot_platform
@@ -16,10 +16,10 @@
     simulation="${simulation}"
     has_arm="true"
-    event_based_sim="${event_based_sim}"
+    simulation_sync="${simulation_sync}"
   />
   <xacro:flying_arm_2
     simulation="${simulation}"
     base_link_name="borinot__base_link"
-    event_based_sim="${event_based_sim}"
+    simulation_sync="${simulation_sync}"
   />
   <gazebo>
@@ -35,8 +35,8 @@
   </gazebo>
   <xacro:if value="${simulation}">
-    <xacro:if value="${event_based_sim}">
+    <xacro:if value="${simulation_sync}">
       <gazebo>
         <plugin name='eagle_gazebo_event_base_sim_plugin'
-          filename='libeagle_gazebo_event_based_sim_plugin.so'>
+          filename='libeagle_gazebo_simulation_sync_plugin.so'>
           <simulationRate>2000</simulationRate>
           <actuationRate>500</actuationRate>

File: robots/common/xacro/multicopter.xacro (robot description, xacro)
@@ -27,5 +27,5 @@
   </xacro:macro>
   <xacro:macro name="rotor"
-    params="platform_name rotor_number parent_link x y z direction simulation event_based_sim">
+    params="platform_name rotor_number parent_link x y z direction simulation simulation_px4">
     <xacro:property name="link_name" value="${platform_name}__rotor${rotor_number}" />
     <xacro:property name="joint_name" value="${platform_name}__j_rotor${rotor_number}" />
@@ -70,5 +70,6 @@
     </joint>
     <xacro:if value="${simulation}">
-      <xacro:unless value="${event_based_sim}">
+      <!-- I should check also here simulation_sync, for safety -->
+      <xacro:if value="${simulation_px4}">
         <gazebo>
           <plugin name='${joint_name}_plugin' filename='libgazebo_motor_model.so'>
@@ -90,5 +91,5 @@
           </plugin>
         </gazebo>
-      </xacro:unless>
+      </xacro:if>
     </xacro:if>
   </xacro:macro>

File: robots/flying_arm_2/xacro/definition.urdf.xacro (robot description, xacro)
@@ -1,4 +1,4 @@
 <robot xmlns:xacro="http://www.ros.org/wiki/xacro">
-  <xacro:macro name="flying_arm_2" params="simulation event_based_sim base_link_name">
+  <xacro:macro name="flying_arm_2" params="simulation simulation_sync base_link_name">
     <xacro:property name="platform_name" value="borinot" />
     <xacro:if value="${base_link_name==''}">
@@ -101,5 +101,5 @@
     </joint>
     <xacro:if value="${simulation}">
-      <xacro:unless value="${event_based_sim}">
+      <xacro:unless value="${simulation_sync}">
         <gazebo>
           <plugin name="odri_gazebo" filename="libodri_gazebo_plugin.so">
