Commit message: wip

File: robots/borinot/xacro/description.urdf.xacro (robot description, xacro)
@@ -15,9 +15,10 @@
   <xacro:property name="simulation_sync" value="$(arg simulation_sync)" />
   <xacro:property name="simulation_px4" value="$(arg simulation_px4)" />
+  <xacro:property name="robot_name" value="borinot" />
   <xacro:if value="${simulation_sync}">
     <xacro:property name="simulation_px4" value="false" />
   </xacro:if>
   <xacro:borinot_platform
-    robot_name="borinot"
+    robot_name="${robot_name}"
     simulation="${simulation}"
     simulation_sync="${simulation_sync}"
@@ -32,6 +33,6 @@
           <simulationRate>2000</simulationRate>
           <actuationRate>500</actuationRate>
-          <ramStateTopic>/borinot/ram_state</ramStateTopic>
-          <ramControlTopic>/borinot/ram_control</ramControlTopic>
+          <ramStateTopic>/${robot_name}/ram_state</ramStateTopic>
+          <ramControlTopic>/${robot_name}/ram_control</ramControlTopic>
           <platform_params>
             <baselinkName>borinot__base_link</baselinkName>
@@ -77,5 +78,5 @@
           <plugin name='eagle_ros2_gz::EagleGzRamStateSensorPlugin'
             filename='libeagle_gz_ram_state_sensor_plugin.so'>
-            <ramStateTopic>/borinot/ram_state</ramStateTopic>
+            <ramStateTopic>/${robot_name}/ram_state</ramStateTopic>
             <platform_params>
               <linkName>borinot__base_link</linkName>
@@ -84,5 +85,5 @@
           <plugin name='eagle_ros2_gz::EagleGzRamFtControllerPlugin'
             filename='libeagle_gz_ram_ft_controller_plugin.so'>
-            <ramControlTopic>/borinot/ram_control</ramControlTopic>
+            <ramControlTopic>/${robot_name}/ram_control</ramControlTopic>
             <platform_params>
               <linkName>borinot__base_link</linkName>

File: robots/borinot_flying_arm_2/xacro/description.urdf.xacro (robot description, xacro)
@@ -8,13 +8,19 @@
   <xacro:arg name="simulation" default="true" />
   <xacro:arg name="simulation_sync" default="false" />
+  <xacro:arg name="simulation_px4" default="false" />
   <!-- properties -->
   <xacro:property name="simulation" value="$(arg simulation)" />
   <xacro:property name="simulation_sync" value="$(arg simulation_sync)" />
+  <xacro:property name="simulation_px4" value="$(arg simulation_px4)" />
   <xacro:property name="robot_name" value="borinot_flying_arm_2" />
+  <xacro:if value="${simulation_sync}">
+    <xacro:property name="simulation_px4" value="false" />
+  </xacro:if>
   <xacro:borinot_platform
     robot_name="${robot_name}"
     simulation="${simulation}"
+    simulation_sync="${simulation_sync}"
+    simulation_px4="${simulation_px4}"
     has_arm="true"
-    simulation_sync="${simulation_sync}"
   />
   <xacro:flying_arm_2
@@ -23,24 +29,13 @@
     simulation_sync="${simulation_sync}"
   />
-  <gazebo>
-    <plugin name='external_force_plugin' filename='libeagle_gazebo_force_plugin.so'>
-      <namespace>${robot_name}</namespace>
-      <trajectoryName>aasquare.yaml</trajectoryName>
-      <linkName>borinot__base_link</linkName>
-      <direction>1 0 0</direction>
-      <instant>1.0</instant>
-      <magnitude>30.0</magnitude>
-      <duration>1.0</duration>
-    </plugin>
-  </gazebo>
   <xacro:if value="${simulation}">
     <xacro:if value="${simulation_sync}">
       <gazebo>
-        <plugin name='eagle_gazebo_event_base_sim_plugin'
-          filename='libeagle_gazebo_simulation_sync_plugin.so'>
+        <plugin name='eagle_ros2_gz::EagleGzSyncSimPlugin'
+          filename='libeagle_gz_sync_sim_plugin.so'>
           <simulationRate>2000</simulationRate>
           <actuationRate>500</actuationRate>
-          <uamStateTopic>/${robot_name}/uam_state</uamStateTopic>
-          <uamControlTopic>/${robot_name}/uam_control</uamControlTopic>
+          <ramStateTopic>/${robot_name}/uam_state</ramStateTopic>
+          <ramControlTopic>/${robot_name}/uam_control</ramControlTopic>
           <platform_params>
             <baselinkName>borinot__base_link</baselinkName>
@@ -90,4 +85,56 @@
       </gazebo>
     </xacro:if>
+    <xacro:unless value="${simulation_sync}">
+      <xacro:unless value="${simulation_px4}">
+        <gazebo>
+          <plugin name='eagle_ros2_gz::EagleGzRamStateSensorPlugin'
+            filename='libeagle_gz_ram_state_sensor_plugin.so'>
+            <ramStateTopic>/${robot_name}/ram_state</ramStateTopic>
+            <platform_params>
+              <linkName>borinot__base_link</linkName>
+            </platform_params>
+          </plugin>
+          <plugin name='eagle_ros2_gz::EagleGzRamFtControllerPlugin'
+            filename='libeagle_gz_ram_ft_controller_plugin.so'>
+            <ramControlTopic>/${robot_name}/ram_control</ramControlTopic>
+            <platform_params>
+              <linkName>borinot__base_link</linkName>
+              <thrustToTorqueRatio>0.016894178436859097</thrustToTorqueRatio>
+              <thrustBias>1.0</thrustBias>
+              <rotor_params>
+                <number>0</number>
+                <linkName>borinot__rotor0</linkName>
+                <turningDirection>-1</turningDirection>
+              </rotor_params>
+              <rotor_params>
+                <number>1</number>
+                <linkName>borinot__rotor1</linkName>
+                <turningDirection>1</turningDirection>
+              </rotor_params>
+              <rotor_params>
+                <number>2</number>
+                <linkName>borinot__rotor2</linkName>
+                <turningDirection>-1</turningDirection>
+              </rotor_params>
+              <rotor_params>
+                <number>3</number>
+                <linkName>borinot__rotor3</linkName>
+                <turningDirection>1</turningDirection>
+              </rotor_params>
+              <rotor_params>
+                <number>4</number>
+                <linkName>borinot__rotor4</linkName>
+                <turningDirection>1</turningDirection>
+              </rotor_params>
+              <rotor_params>
+                <number>5</number>
+                <linkName>borinot__rotor5</linkName>
+                <turningDirection>-1</turningDirection>
+              </rotor_params>
+            </platform_params>
+          </plugin>
+        </gazebo>
+      </xacro:unless>
+    </xacro:unless>
   </xacro:if>
 </robot>
