Commit message: fix (bfa2): add parameters to use the arm

File: robots/borinot_flying_arm_2/xacro/description.urdf.xacro (robot description, xacro)
@@ -26,6 +26,7 @@
   <xacro:flying_arm_2
     simulation="${simulation}"
+    simulation_sync="${simulation_sync}"
+    simulation_px4="${simulation_px4}"
     base_link_name="borinot__base_link"
-    simulation_sync="${simulation_sync}"
   />
   <xacro:if value="${simulation}">
@@ -94,4 +95,14 @@
               <linkName>borinot__base_link</linkName>
             </platform_params>
+            <arm_params>
+              <joint_params>
+                <number>0</number>
+                <jointName>flying_arm_2__j_bl_link1</jointName>
+              </joint_params>
+              <joint_params>
+                <number>1</number>
+                <jointName>flying_arm_2__j_link1_link2</jointName>
+              </joint_params>
+            </arm_params>
           </plugin>
           <plugin name='eagle_ros2_gz::EagleGzRamFtControllerPlugin'
@@ -133,4 +144,14 @@
               </rotor_params>
             </platform_params>
+            <arm_params>
+              <joint_params>
+                <number>0</number>
+                <jointName>flying_arm_2__j_bl_link1</jointName>
+              </joint_params>
+              <joint_params>
+                <number>1</number>
+                <jointName>flying_arm_2__j_link1_link2</jointName>
+              </joint_params>
+            </arm_params>
           </plugin>
         </gazebo>

File: robots/flying_arm_2/xacro/definition.urdf.xacro (robot description, xacro)
@@ -1,4 +1,4 @@
 <robot xmlns:xacro="http://www.ros.org/wiki/xacro">
-  <xacro:macro name="flying_arm_2" params="simulation simulation_sync base_link_name">
+  <xacro:macro name="flying_arm_2" params="simulation simulation_sync simulation_px4 base_link_name">
     <xacro:property name="platform_name" value="borinot" />
     <xacro:if value="${base_link_name==''}">
@@ -101,5 +101,5 @@
     </joint>
     <xacro:if value="${simulation}">
-      <xacro:unless value="${simulation_sync}">
+      <xacro:if value="${simulation_px4}">
         <gazebo>
           <plugin name="odri_gazebo" filename="libodri_gazebo_plugin.so">
@@ -118,5 +118,5 @@
           </plugin>
         </gazebo>
-      </xacro:unless>
+      </xacro:if>
     </xacro:if>
   </xacro:macro>
